File: HV_stepstick_adapter.sch (KiCad schematic (older format))
At the start: 5 parts, among them J1 Screw_Terminal_01x02, J2 Conn_01x08, J3 Conn_01x08, J4 Conn_01x02

Commit message: Added diode for safety
Added a Schottky diode between VDD and VMOT lines for safety; also slightly reduced PCB width, to improve the fit on boards; and now Gerber files are available.
Parts:
- added D1: MBR1100G, Diode_THT:D_DO-41_SOD81_P10.16mm_Horizontal, symbol Device:D
Connections:
- net VDD: now also D1.2 (A)
- net VMOT: now also D1.1 (K)
Changed lines of the file:
@@
 Text GLabel 2250 3300 0    39   Input ~ 0
 DIR
+$Comp
+L Device:D D1
+U 1 1 61B2076B
+P 3300 3050
+F 0 "D1" H 3300 2833 50  0000 C CNN
+F 1 "MBR1100G" H 3300 2924 50  0000 C CNN
+F 2 "Diode_THT:D_DO-41_SOD81_P10.16mm_Horizontal" H 3300 3050 50  0001 C CNN
+F 3 "~" H 3300 3050 50  0001 C CNN
+	1    3300 3050
+	-1   0    0    1
+$EndComp
+Wire Wire Line
+	3500 3050 3450 3050
+Text GLabel 3500 3050 2    39   Input ~ 0
+VMOT
+$Comp
+L power:VDD #PWR0101
+U 1 1 61B21D06
+P 3000 3050
+F 0 "#PWR0101" H 3000 2900 50  0001 C CNN
+F 1 "VDD" H 2900 3200 50  0000 L CNN
+F 2 "" H 3000 3050 50  0001 C CNN
+F 3 "" H 3000 3050 50  0001 C CNN
+	1    3000 3050
+	1    0    0    -1
+$EndComp
+Wire Wire Line
+	3000 3050 3150 3050
 $EndSCHEMATC
